File: design/LattePanda_DriverStation/lattepanda_driverstation.brd (EAGLE design)
At the start: 18 parts, among them CN1 0.1, CN2 0.1, CN3 0.1, CN4 0.1, IC1 MCP23017SS, U1 PCA9685

Commit message: Progress commit.
Parts:
- added C3: 0.1, rcl:C1206
- added D1, D2, D3, D4, D5: (no value), SparkFun-LED:LED-1206
- added IC4: PCA9685, SparkFun-DigitalIC:TSSOP-28_4MM
- added Q1, Q2: MOSFET-NCHANNELAO3404A, SparkFun-DiscreteSemi:SOT23-3
- added R10, R11, R12, R13, R14: (no value), rcl:M1206
- added R15, R16, R9: 220, SparkFun-Resistors:0603-ARV
- R8: value (none) -> 220; device rcl:M1206 -> SparkFun-Resistors:0603-ARV
- moved R8 106.3 mm to (-73.7, -148.6)
- renumbered U$1 to J1, U$3 to IC2, U1 to IC3
Connections:
- removed net PWM_OE_N: J1.D11
- new net DIO0: IC1.21
- new net DIO1: IC1.22
- new net DIO10: IC1.3
- new net DIO11: IC1.4
- new net DIO12: IC1.5
- new net DIO13: IC1.6
- new net DIO14: IC1.7
- new net DIO15: IC1.8
- new net DIO2: IC1.23
- new net DIO3: IC1.24
- new net DIO4: IC1.25
- new net DIO5: IC1.26
- new net DIO6: IC1.27
- new net DIO7: IC1.28
- new net DIO8: IC1.1
- new net DIO9: IC1.2
- new net ENABLE_IO: IC1.18, IC2.15, IC3.23, IC4.23, J1.D12
- new net LED_CH0: R8.1
- new net LED_CH1: R8.2
- new net LED_CH10: R16.6
- new net LED_CH11: R16.5
- new net LED_CH12: R15.8
- new net LED_CH13: R15.7
- new net LED_CH14: R15.6
- new net LED_CH15: R15.5
- new net LED_CH2: R8.3
- new net LED_CH3: R8.4
- new net LED_CH4: R9.1
- new net LED_CH5: R9.2
- new net LED_CH6: R9.3
- new net LED_CH7: R9.4
- new net LED_CH8: R16.8
- new net LED_CH9: R16.7
- new net N$18: IC4.7, R8.7
- new net N$19: D1.A
- new net N$20: D2.A
- new net N$21: D3.A
- new net N$22: D4.A
- new net N$23: D5.A
- new net N$24: IC4.8, R8.6
- new net N$25: IC4.9, R8.5
- new net N$26: IC4.10, R9.8
- new net N$27: IC4.11, R9.7
- new net N$28: IC4.12, R9.6
- new net N$29: IC4.13, R9.5
- new net N$30: IC4.15, R15.4
- new net N$31: IC4.16, R15.3
- new net N$32: IC4.17, R15.2
- new net N$33: IC4.18, R15.1
- new net N$34: IC4.19, R16.4
- new net N$35: IC4.20, R16.3
- new net N$36: IC4.21, R16.2
- new net N$37: IC4.22, R16.1
- new net STATUS_LED: J1.D13
- net +5V: now also C3.1, IC4.28
- net ANA_MUX_COM: now also J1.A5; no longer J1.A3
- net ANA_MUX_S0: no longer J1.D4
- net ANA_MUX_S1: no longer J1.D5
- net ANA_MUX_S2: no longer J1.D6
- net ANA_MUX_S3: no longer J1.D8
- net GND: now also C3.2, IC4.14; no longer R8.1
- net I2C_SCL: now also IC4.26
- net I2C_SDA: now also IC4.27
- net N$17: now also IC4.6, R8.8; no longer IC2.15, R8.2

Commit message: 
Parts:
- removed CN1, CN2, CN3, CN4: 0.1, resistor-dil:EXB38V
- removed R15, R16, R9: 220, SparkFun-Resistors:0603-ARV
- added C4, C5, C6, C8: 0.1, rcl:C1206
- added IC5, IC6, IC7: ADS1015, SparkFun-AnalogIC:MSOP10
- added J2: (no value), SparkFun-Connectors:1X04
- added J3: TEMP_SENSE, SparkFun-Connectors:MOLEX-1X3_LOCK
- added J4: FAN_OUT, SparkFun-Connectors:MOLEX-1X3_LOCK
- added U$1: ANALOGHEADER, ControlBoard:ANALOGHEADER
- added U$2: DIGITALOUTPUTS, ControlBoard:DIGITALOUT
- IC2: value MUX-74HC4067SMD -> PCA9685; device SparkFun-AnalogIC:SSOP24 -> SparkFun-DigitalIC:TSSOP-28_4MM
- IC3: value PCA9685 -> TLC59116; device SparkFun-DigitalIC:TSSOP-28_4MM -> TI_TLC59116:TSSOP28
- IC4: value PCA9685 -> ADS1015; device SparkFun-DigitalIC:TSSOP-28_4MM -> SparkFun-AnalogIC:MSOP10
- R8: value 220 -> (none); device SparkFun-Resistors:0603-ARV -> rcl:R1206
- moved C2 172.4 mm to (-109.2, -201.9), turned to 90 degrees
- moved IC3 166.3 mm to (-111.8, -152.4), turned to 180 degrees
- moved R7 121.5 mm to (8.89, 76.2), turned to 270 degrees
- moved R6 113.3 mm to (8.89, 72.4), turned to 270 degrees
- moved R5 97.9 mm to (8.89, 58.4), turned to 90 degrees
- moved R4 96.1 mm to (8.89, 62.2), turned to 90 degrees
- moved IC4 72.6 mm to (-115.6, -191.8), turned to 180 degrees
- moved IC1 59.4 mm to (19.1, 49.5)
- moved IC2 58.5 mm to (19.1, 67.3), turned to 270 degrees
- moved C3 31.4 mm to (-102.9, -153.7), turned to 90 degrees
- moved R8 29.2 mm to (-102.9, -147.3), turned to 180 degrees
Connections:
- net DIO0 renamed DIO_CH0
- net DIO1 renamed DIO_CH1
- net DIO10 renamed DIO_CH10
- net DIO11 renamed DIO_CH11
- net DIO12 renamed DIO_CH12
- net DIO13 renamed DIO_CH13
- net DIO14 renamed DIO_CH14
- net DIO15 renamed DIO_CH15
- net DIO2 renamed DIO_CH2
- net DIO3 renamed DIO_CH3
- net DIO4 renamed DIO_CH4
- net DIO5 renamed DIO_CH5
- net DIO6 renamed DIO_CH6
- net DIO7 renamed DIO_CH7
- net DIO8 renamed DIO_CH8
- net DIO9 renamed DIO_CH9
- removed net ANA_MUX_COM: IC2.1, J1.A5
- removed net ANA_MUX_S0: IC2.10
- removed net ANA_MUX_S1: IC2.11
- removed net ANA_MUX_S2: IC2.14
- removed net ANA_MUX_S3: IC2.13
- removed net N$18: IC4.7, R8.7
- removed net N$24: IC4.8, R8.6
- removed net N$25: IC4.9, R8.5
- removed net N$26: IC4.10, R9.8
- removed net N$27: IC4.11, R9.7
- removed net N$28: IC4.12, R9.6
- removed net N$29: IC4.13, R9.5
- removed net N$30: IC4.15, R15.4
- removed net N$31: IC4.16, R15.3
- removed net N$32: IC4.17, R15.2
- removed net N$33: IC4.18, R15.1
- removed net N$34: IC4.19, R16.4
- removed net N$35: IC4.20, R16.3
- removed net N$36: IC4.21, R16.2
- removed net N$37: IC4.22, R16.1
- net +5V: now also C4.1, C5.1, C6.1, C8.1, IC2.28, IC4.8, IC5.1, IC5.8, IC6.8, IC7.8, J2.2, U$1.+5V@0, U$1.+5V@1, U$1.+5V@10, U$1.+5V@11, U$1.+5V@12, U$1.+5V@13, U$1.+5V@14, U$1.+5V@15, U$1.+5V@2, U$1.+5V@3, U$1.+5V@4, U$1.+5V@5, U$1.+5V@6, U$1.+5V@7, U$1.+5V@8, U$1.+5V@9, U$2.+5V@0, U$2.+5V@1, U$2.+5V@10, U$2.+5V@11, U$2.+5V@12, U$2.+5V@13, U$2.+5V@14, U$2.+5V@15, U$2.+5V@2, U$2.+5V@3, U$2.+5V@4, U$2.+5V@5, U$2.+5V@6, U$2.+5V@7, U$2.+5V@8, U$2.+5V@9; no longer IC2.24, IC4.28
- net ANA_CH0: now also IC4.4, U$1.0; no longer CN1.1, IC2.9
- net ANA_CH1: now also IC4.5, U$1.1; no longer CN1.2, IC2.8
- net ANA_CH10: now also IC6.6, U$1.10; no longer CN3.3, IC2.21
- net ANA_CH11: now also IC6.7, U$1.11; no longer CN3.4, IC2.20
- net ANA_CH12: now also IC7.4, U$1.12; no longer CN4.1, IC2.19
- net ANA_CH13: now also IC7.5, U$1.13; no longer CN4.2, IC2.18
- net ANA_CH14: now also IC7.6, U$1.14; no longer CN4.3, IC2.17
- net ANA_CH15: now also IC7.7, U$1.15; no longer CN4.4, IC2.16
- net ANA_CH2: now also IC4.6, U$1.2; no longer CN1.3, IC2.7
- net ANA_CH3: now also IC4.7, U$1.3; no longer CN1.4, IC2.6
- net ANA_CH4: now also IC5.4, U$1.4; no longer CN2.1, IC2.5
- net ANA_CH5: now also IC5.5, U$1.5; no longer CN2.2, IC2.4
- net ANA_CH6: now also IC5.6, U$1.6; no longer CN2.3, IC2.3
- net ANA_CH7: now also IC5.7, U$1.7; no longer CN2.4, IC2.2
- net ANA_CH8: now also IC6.4, U$1.8; no longer CN3.1, IC2.23
- net ANA_CH9: now also IC6.5, U$1.9; no longer CN3.2, IC2.22
- net ENABLE_IO: now also IC2.23, IC3.25; no longer IC2.15, IC3.23, IC4.23
- net GND: now also C4.2, C5.2, C6.2, C8.2, IC2.14, IC3.10, IC3.19, IC3.24, IC4.1, IC4.3, IC5.3, IC6.3, IC7.3, J2.1, R8.1, U$1.GND@0, U$1.GND@1, U$1.GND@10, U$1.GND@11, U$1.GND@12, U$1.GND@13, U$1.GND@14, U$1.GND@15, U$1.GND@2, U$1.GND@3, U$1.GND@4, U$1.GND@5, U$1.GND@6, U$1.GND@7, U$1.GND@8, U$1.GND@9; no longer CN1.5, CN1.6, CN1.7, CN1.8, CN2.5, CN2.6, CN2.7, CN2.8, CN3.5, CN3.6, CN3.7, CN3.8, CN4.5, CN4.6, CN4.7, CN4.8, IC2.12, IC3.14, IC4.14
- net I2C_SCL: now also IC2.26, IC4.10, IC5.10, IC6.10, IC7.1, IC7.10, J2.4; no longer IC4.26
- net I2C_SDA: now also IC2.27, IC4.9, IC5.9, IC6.1, IC6.9, IC7.9, J2.3; no longer IC4.27
- net LED_CH0: now also IC3.6, U$2.DO0; no longer R8.1
- net LED_CH1: now also IC3.7, U$2.DO1; no longer R8.2
- net LED_CH10: now also IC3.17, U$2.DO10; no longer R16.6
- net LED_CH11: now also IC3.18, U$2.DO11; no longer R16.5
- net LED_CH12: now also IC3.20, U$2.DO12; no longer R15.8
- net LED_CH13: now also IC3.21, U$2.DO13; no longer R15.7
- net LED_CH14: now also IC3.22, U$2.DO14; no longer R15.6
- net LED_CH15: now also IC3.23, U$2.DO15; no longer R15.5
- net LED_CH2: now also IC3.8, U$2.DO2; no longer R8.3
- net LED_CH3: now also IC3.9, U$2.DO3; no longer R8.4
- net LED_CH4: now also IC3.11, U$2.DO4; no longer R9.1
- net LED_CH5: now also IC3.12, U$2.DO5; no longer R9.2
- net LED_CH6: now also IC3.13, U$2.DO6; no longer R9.3
- net LED_CH7: now also IC3.14, U$2.DO7; no longer R9.4
- net LED_CH8: now also IC3.15, U$2.DO8; no longer R16.8
- net LED_CH9: now also IC3.16, U$2.DO9; no longer R16.7
- net N$1: now also IC2.6; no longer IC3.6
- net N$10: now also IC2.16; no longer IC3.16
- net N$11: now also IC2.17; no longer IC3.17
- net N$12: now also IC2.18; no longer IC3.18
- net N$13: now also IC2.19; no longer IC3.19
- net N$14: now also IC2.20; no longer IC3.20
- net N$15: now also IC2.21; no longer IC3.21
- net N$16: now also IC2.22; no longer IC3.22
- net N$17: now also IC3.1, R8.2; no longer IC4.6, R8.8
- net N$2: now also IC2.7; no longer IC3.7
- net N$3: now also IC2.8; no longer IC3.8
- net N$4: now also IC2.9; no longer IC3.9
- net N$5: now also IC2.10; no longer IC3.10
- net N$6: now also IC2.11; no longer IC3.11
- net N$7: now also IC2.12; no longer IC3.12
- net N$8: now also IC2.13; no longer IC3.13
- net N$9: now also IC2.15; no longer IC3.15

Commit message: 
Parts:
- moved C6 295.5 mm to (52.1, 25.4), turned to 180 degrees
- moved IC7 293.8 mm to (52.1, 19.1), turned to 270 degrees
- moved C5 281.5 mm to (41.9, 25.4), turned to 180 degrees
- moved IC6 279.7 mm to (41.9, 19.1), turned to 270 degrees
- moved C2 267.5 mm to (31.8, 25.4), turned to 180 degrees
- moved IC5 265.6 mm to (31.8, 19.1), turned to 270 degrees
- moved C8 253.5 mm to (21.6, 25.4), turned to 180 degrees
- moved IC3 252.2 mm to (39.4, 49.5), turned to 270 degrees
- moved IC4 251.5 mm to (21.6, 19.1), turned to 270 degrees
- moved U$2 247.2 mm to (35.6, 39.4), turned to 0 degrees
- moved U$1 229.3 mm to (6.35, 15.2), turned to 270 degrees
- moved IC1 50.8 mm to (62.2, 76.2)
- moved R7 29.9 mm to (38.1, 69.8)
- moved R4 29.9 mm to (38.1, 55.9)
- moved R5 29.9 mm to (38.1, 52.1)
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Routing:
- net LED_CH15: track 0.00 -> 20.2 mm
- net LED_CH0: track 0.00 -> 20.2 mm
- net LED_CH14: track 0.00 -> 17.4 mm
- net LED_CH1: track 0.00 -> 17.4 mm
- net LED_CH13: track 0.00 -> 14.6 mm
- net LED_CH2: track 0.00 -> 14.6 mm
- net LED_CH12: track 0.00 -> 12.5 mm
- net LED_CH3: track 0.00 -> 12.5 mm
- net LED_CH11: track 0.00 -> 10.2 mm
- net LED_CH4: track 0.00 -> 10.2 mm
- net LED_CH10: track 0.00 -> 8.13 mm
- net LED_CH5: track 0.00 -> 8.13 mm
- net LED_CH9: track 0.00 -> 6.07 mm
- net LED_CH6: track 0.00 -> 6.07 mm
- net ANA_CH3: track 0.00 -> 5.89 mm
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