File: design/LattePanda_DriverStation/lattepanda_driverstation.sch (EAGLE design)
At the start: 4 parts

Commit message: Progress made on the schematic.
Parts:
- added C1, C2: 0.1, rcl:C-USC1206
- added CN1, CN2, CN3, CN4: 0.1, resistor-dil:4R-NEXB38V
- added IC1: MCP23017SS, microchip:MCP23017SS
- added R4, R5, R6, R7: 1k, SparkFun-Resistors:RESISTOR-ARRAY0603-ARV
- added R8: (no value), rcl:R-US_M1206
- added U$3: MUX-74HC4067SMD, SparkFun-AnalogIC:MUX-74HC4067SMD
- added U1: PCA9685, SparkFun-DigitalIC:PCA9685
Connections:
- new net ANA_CH0: CN1A.1, U$3.CHAN0
- new net ANA_CH1: CN1B.1, U$3.CHAN1
- new net ANA_CH10: CN3C.1, U$3.CHAN10
- new net ANA_CH11: CN3D.1, U$3.CHAN11
- new net ANA_CH12: CN4A.1, U$3.CHAN12
- new net ANA_CH13: CN4B.1, U$3.CHAN13
- new net ANA_CH14: CN4C.1, U$3.CHAN14
- new net ANA_CH15: CN4D.1, U$3.CHAN15
- new net ANA_CH2: CN1C.1, U$3.CHAN2
- new net ANA_CH3: CN1D.1, U$3.CHAN3
- new net ANA_CH4: CN2A.1, U$3.CHAN4
- new net ANA_CH5: CN2B.1, U$3.CHAN5
- new net ANA_CH6: CN2C.1, U$3.CHAN6
- new net ANA_CH7: CN2D.1, U$3.CHAN7
- new net ANA_CH8: CN3A.1, U$3.CHAN8
- new net ANA_CH9: CN3B.1, U$3.CHAN9
- new net ANA_MUX_COM: U$1.A3, U$3.COM
- new net N$10: R4C.1, U1.CH9
- new net N$11: R4B.1, U1.CH10
- new net N$12: R4A.1, U1.CH11
- new net N$13: R5D.1, U1.CH12
- new net N$14: R5C.1, U1.CH13
- new net N$15: R5B.1, U1.CH14
- new net N$16: R5A.1, U1.CH15
- new net N$17: R8.2, U$3.EN
- new net N$2: R7B.2, U1.CH1
- new net N$3: R7C.2, U1.CH2
- new net N$4: R7D.2, U1.CH3
- new net N$5: R6A.2, U1.CH4
- new net N$6: R6B.2, U1.CH5
- new net N$7: R6C.2, U1.CH6
- new net N$8: R6D.2, U1.CH7
- new net N$9: R4D.1, U1.CH8
- new net PWM_CH0: R7A.1
- new net PWM_CH1: R7B.1
- new net PWM_CH10: R4B.2
- new net PWM_CH11: R4A.2
- new net PWM_CH12: R5D.2
- new net PWM_CH13: R5C.2
- new net PWM_CH14: R5B.2
- new net PWM_CH15: R5A.2
- new net PWM_CH2: R7C.1
- new net PWM_CH3: R7D.1
- new net PWM_CH4: R6A.1
- new net PWM_CH5: R6B.1
- new net PWM_CH6: R6C.1
- new net PWM_CH7: R6D.1
- new net PWM_CH8: R4D.2
- new net PWM_CH9: R4C.2
- net +5V: now also C1.1, C2.1, IC1.VDD, U$3.VCC, U1.VDD
- net ANA_MUX_S0: now also U$3.S0
- net ANA_MUX_S1: now also U$3.S1
- net ANA_MUX_S2: now also U$3.S2
- net ANA_MUX_S3: now also U$3.S3
- net GND: now also C1.2, C2.2, CN1A.2, CN1B.2, CN1C.2, CN1D.2, CN2A.2, CN2B.2, CN2C.2, CN2D.2, CN3A.2, CN3B.2, CN3C.2, CN3D.2, CN4A.2, CN4B.2, CN4C.2, CN4D.2, IC1.VSS, R8.1, U$3.GND, U1.VSS
- net I2C_SCL: now also IC1.SCL, U1.SCL
- net I2C_SDA: now also IC1.SDA, U1.SDA
- net N$1: now also R7A.2, U1.CH0; no longer U$1.A3

Commit message: Progress commit.
Parts:
- added C3: 0.1, rcl:C-USC1206
- added D1, D2, D3, D4, D5: (no value), SparkFun-LED:LED1206
- added IC4: PCA9685, SparkFun-DigitalIC:PCA9685
- added Q1, Q2: MOSFET-NCHANNELAO3404A, SparkFun-DiscreteSemi:MOSFET-NCHANNELAO3404A
- added R10, R11, R12, R13, R14: (no value), rcl:R-US_M1206
- added R15, R16, R9: 220, SparkFun-Resistors:RESISTOR-ARRAY0603-ARV
- R8: value (none) -> 220; device rcl:R-US_M1206 -> SparkFun-Resistors:RESISTOR-ARRAY0603-ARV
- renumbered U$1 to J1, U$3 to IC2, U1 to IC3
Connections:
- removed net PWM_OE_N: J1.D11_SHARED
- new net DIO0: IC1.GPA0
- new net DIO1: IC1.GPA1
- new net DIO10: IC1.GPB2
- new net DIO11: IC1.GPB3
- new net DIO12: IC1.GPB4
- new net DIO13: IC1.GPB5
- new net DIO14: IC1.GPB6
- new net DIO15: IC1.GPB7
- new net DIO2: IC1.GPA2
- new net DIO3: IC1.GPA3
- new net DIO4: IC1.GPA4
- new net DIO5: IC1.GPA5
- new net DIO6: IC1.GPA6
- new net DIO7: IC1.GPA7
- new net DIO8: IC1.GPB0
- new net DIO9: IC1.GPB1
- new net ENABLE_IO: IC1.!RESET, IC2.EN, IC3.!OE, IC4.!OE, J1.D12
- new net LED_CH0: R8A.1
- new net LED_CH1: R8B.1
- new net LED_CH10: R16C.2
- new net LED_CH11: R16D.2
- new net LED_CH12: R15A.2
- new net LED_CH13: R15B.2
- new net LED_CH14: R15C.2
- new net LED_CH15: R15D.2
- new net LED_CH2: R8C.1
- new net LED_CH3: R8D.1
- new net LED_CH4: R9A.1
- new net LED_CH5: R9B.1
- new net LED_CH6: R9C.1
- new net LED_CH7: R9D.1
- new net LED_CH8: R16A.2
- new net LED_CH9: R16B.2
- new net N$18: IC4.CH1, R8B.2
- new net N$19: D1.A
- new net N$20: D2.A
- new net N$21: D3.A
- new net N$22: D4.A
- new net N$23: D5.A
- new net N$24: IC4.CH2, R8C.2
- new net N$25: IC4.CH3, R8D.2
- new net N$26: IC4.CH4, R9A.2
- new net N$27: IC4.CH5, R9B.2
- new net N$28: IC4.CH6, R9C.2
- new net N$29: IC4.CH7, R9D.2
- new net N$30: IC4.CH8, R15D.1
- new net N$31: IC4.CH9, R15C.1
- new net N$32: IC4.CH10, R15B.1
- new net N$33: IC4.CH11, R15A.1
- new net N$34: IC4.CH12, R16D.1
- new net N$35: IC4.CH13, R16C.1
- new net N$36: IC4.CH14, R16B.1
- new net N$37: IC4.CH15, R16A.1
- new net STATUS_LED: J1.D13
- net +5V: now also C3.1, IC4.VDD
- net ANA_MUX_COM: now also J1.A5; no longer J1.A3
- net ANA_MUX_S0: no longer J1.D4
- net ANA_MUX_S1: no longer J1.D5
- net ANA_MUX_S2: no longer J1.D6
- net ANA_MUX_S3: no longer J1.D8
- net GND: now also C3.2, IC4.VSS; no longer R8.1
- net I2C_SCL: now also IC4.SCL
- net I2C_SDA: now also IC4.SDA
- net N$17: now also IC4.CH0, R8A.2; no longer IC2.EN, R8.2
Other:
- note added: "BATTERY_CHARGED"
- note added: "BATTERY_CHARGING"
- note added: "EXTERNAL_POWER_GOOD"
- note added: "OUTPUTS_ENABLED"
- note added: "STATUS_LED"
- moved on the sheet: R4A, R4B, R4C, R4D, R5A, R5B, R5C, R5D

Commit message: 
Parts:
- removed CN1, CN2, CN3, CN4: 0.1, resistor-dil:4R-NEXB38V
- removed R15, R16, R9: 220, SparkFun-Resistors:RESISTOR-ARRAY0603-ARV
- added C4, C5, C6, C8: 0.1, rcl:C-USC1206
- added IC5, IC6, IC7: ADS1015, SparkFun-AnalogIC:ADS1015
- added J2: (no value), SparkFun-Connectors:I2C_STANDARD
- added J3: TEMP_SENSE, SparkFun-Connectors:M03POLAR_LOCK
- added J4: FAN_OUT, SparkFun-Connectors:M03POLAR_LOCK
- added U$1: ANALOGHEADER, ControlBoard:ANALOGHEADER
- added U$2: DIGITALOUTPUTS, ControlBoard:DIGITALOUTPUTS
- IC2: value MUX-74HC4067SMD -> PCA9685; device SparkFun-AnalogIC:MUX-74HC4067SMD -> SparkFun-DigitalIC:PCA9685
- IC3: value PCA9685 -> TLC59116; device SparkFun-DigitalIC:PCA9685 -> TI_TLC59116:TLC59116
- IC4: value PCA9685 -> ADS1015; device SparkFun-DigitalIC:PCA9685 -> SparkFun-AnalogIC:ADS1015
- R8: value 220 -> (none); device SparkFun-Resistors:RESISTOR-ARRAY0603-ARV -> rcl:R-US_R1206
Connections:
- net DIO0 renamed DIO_CH0
- net DIO1 renamed DIO_CH1
- net DIO10 renamed DIO_CH10
- net DIO11 renamed DIO_CH11
- net DIO12 renamed DIO_CH12
- net DIO13 renamed DIO_CH13
- net DIO14 renamed DIO_CH14
- net DIO15 renamed DIO_CH15
- net DIO2 renamed DIO_CH2
- net DIO3 renamed DIO_CH3
- net DIO4 renamed DIO_CH4
- net DIO5 renamed DIO_CH5
- net DIO6 renamed DIO_CH6
- net DIO7 renamed DIO_CH7
- net DIO8 renamed DIO_CH8
- net DIO9 renamed DIO_CH9
- removed net ANA_MUX_COM: IC2.COM, J1.A5
- removed net ANA_MUX_S0: IC2.S0
- removed net ANA_MUX_S1: IC2.S1
- removed net ANA_MUX_S2: IC2.S2
- removed net ANA_MUX_S3: IC2.S3
- removed net N$18: IC4.CH1, R8B.2
- removed net N$24: IC4.CH2, R8C.2
- removed net N$25: IC4.CH3, R8D.2
- removed net N$26: IC4.CH4, R9A.2
- removed net N$27: IC4.CH5, R9B.2
- removed net N$28: IC4.CH6, R9C.2
- removed net N$29: IC4.CH7, R9D.2
- removed net N$30: IC4.CH8, R15D.1
- removed net N$31: IC4.CH9, R15C.1
- removed net N$32: IC4.CH10, R15B.1
- removed net N$33: IC4.CH11, R15A.1
- removed net N$34: IC4.CH12, R16D.1
- removed net N$35: IC4.CH13, R16C.1
- removed net N$36: IC4.CH14, R16B.1
- removed net N$37: IC4.CH15, R16A.1
- net +5V: now also C4.1, C5.1, C6.1, C8.1, IC2.VDD, IC3.VCC, IC5.ADDR, IC5.VDD, IC6.VDD, IC7.VDD, J2.2, U$1.+5V, U$2.+5V; no longer IC2.VCC, IC3.VDD
- net ANA_CH0: now also IC4.AIN0, U$1.A0; no longer CN1A.1, IC2.CHAN0
- net ANA_CH1: now also IC4.AIN1, U$1.A1; no longer CN1B.1, IC2.CHAN1
- net ANA_CH10: now also IC6.AIN2, U$1.A10; no longer CN3C.1, IC2.CHAN10
- net ANA_CH11: now also IC6.AIN3, U$1.A11; no longer CN3D.1, IC2.CHAN11
- net ANA_CH12: now also IC7.AIN0, U$1.A12; no longer CN4A.1, IC2.CHAN12
- net ANA_CH13: now also IC7.AIN1, U$1.A13; no longer CN4B.1, IC2.CHAN13
- net ANA_CH14: now also IC7.AIN2, U$1.A14; no longer CN4C.1, IC2.CHAN14
- net ANA_CH15: now also IC7.AIN3, U$1.A15; no longer CN4D.1, IC2.CHAN15
- net ANA_CH2: now also IC4.AIN2, U$1.A2; no longer CN1C.1, IC2.CHAN2
- net ANA_CH3: now also IC4.AIN3, U$1.A3; no longer CN1D.1, IC2.CHAN3
- net ANA_CH4: now also IC5.AIN0, U$1.A4; no longer CN2A.1, IC2.CHAN4
- net ANA_CH5: now also IC5.AIN1, U$1.A5; no longer CN2B.1, IC2.CHAN5
- net ANA_CH6: now also IC5.AIN2, U$1.A6; no longer CN2C.1, IC2.CHAN6
- net ANA_CH7: now also IC5.AIN3, U$1.A7; no longer CN2D.1, IC2.CHAN7
- net ANA_CH8: now also IC6.AIN0, U$1.A8; no longer CN3A.1, IC2.CHAN8
- net ANA_CH9: now also IC6.AIN1, U$1.A9; no longer CN3B.1, IC2.CHAN9
- net ENABLE_IO: now also IC2.!OE, IC3./RESET; no longer IC2.EN, IC3.!OE, IC4.!OE
- net GND: now also C4.2, C5.2, C6.2, C8.2, IC2.VSS, IC3.GND@10, IC3.GND@19, IC3.GND@24, IC4.ADDR, IC5.VSS, IC6.VSS, IC7.VSS, J2.1, R8.1, U$1.GND; no longer CN1A.2, CN1B.2, CN1C.2, CN1D.2, CN2A.2, CN2B.2, CN2C.2, CN2D.2, CN3A.2, CN3B.2, CN3C.2, CN3D.2, CN4A.2, CN4B.2, CN4C.2, CN4D.2, IC2.GND, IC3.VSS
- net I2C_SCL: now also IC2.SCL, IC5.SCL, IC6.SCL, IC7.ADDR, IC7.SCL, J2.4
- net I2C_SDA: now also IC2.SDA, IC5.SDA, IC6.ADDR, IC6.SDA, IC7.SDA, J2.3
- net LED_CH0: now also IC3./OUT0, U$2.DO0; no longer R8A.1
- net LED_CH1: now also IC3./OUT1, U$2.DO1; no longer R8B.1
- net LED_CH10: now also IC3./OUT10, U$2.DO10; no longer R16C.2
- net LED_CH11: now also IC3./OUT11, U$2.DO11; no longer R16D.2
- net LED_CH12: now also IC3./OUT12, U$2.DO12; no longer R15A.2
- net LED_CH13: now also IC3./OUT13, U$2.DO13; no longer R15B.2
- net LED_CH14: now also IC3./OUT14, U$2.DO14; no longer R15C.2
- net LED_CH15: now also IC3./OUT15, U$2.DO15; no longer R15D.2
- net LED_CH2: now also IC3./OUT2, U$2.DO2; no longer R8C.1
- net LED_CH3: now also IC3./OUT3, U$2.DO3; no longer R8D.1
- net LED_CH4: now also IC3./OUT4, U$2.DO4; no longer R9A.1
- net LED_CH5: now also IC3./OUT5, U$2.DO5; no longer R9B.1
- net LED_CH6: now also IC3./OUT6, U$2.DO6; no longer R9C.1
- net LED_CH7: now also IC3./OUT7, U$2.DO7; no longer R9D.1
- net LED_CH8: now also IC3./OUT8, U$2.DO8; no longer R16A.2
- net LED_CH9: now also IC3./OUT9, U$2.DO9; no longer R16B.2
- net N$1: now also IC2.CH0; no longer IC3.CH0
- net N$10: now also IC2.CH9; no longer IC3.CH9
- net N$11: now also IC2.CH10; no longer IC3.CH10
- net N$12: now also IC2.CH11; no longer IC3.CH11
- net N$13: now also IC2.CH12; no longer IC3.CH12
- net N$14: now also IC2.CH13; no longer IC3.CH13
- net N$15: now also IC2.CH14; no longer IC3.CH14
- net N$16: now also IC2.CH15; no longer IC3.CH15
- net N$17: now also IC3.REXT, R8.2; no longer IC4.CH0, R8A.2
- net N$2: now also IC2.CH1; no longer IC3.CH1
- net N$3: now also IC2.CH2; no longer IC3.CH2
- net N$4: now also IC2.CH3; no longer IC3.CH3
- net N$5: now also IC2.CH4; no longer IC3.CH4
- net N$6: now also IC2.CH5; no longer IC3.CH5
- net N$7: now also IC2.CH6; no longer IC3.CH6
- net N$8: now also IC2.CH7; no longer IC3.CH7
- net N$9: now also IC2.CH8; no longer IC3.CH8
Other:
- note added: "ADS1015 Address Selection Table ADDR_PIN SLAVE_ADDRESS Ground 1001000 VDD 1001001 SDA 1001010 SCL 1001011"
- moved on the sheet: C1, C2, C3

Commit message: 
Parts:
- removed J3: TEMP_SENSE, SparkFun-Connectors:M03POLAR_LOCK
- removed J4: FAN_OUT, SparkFun-Connectors:M03POLAR_LOCK
Other:
- moved on the sheet: C1, C3, IC2, R4A, R4B, R4C, R4D, R5A, R5B, R5C, R5D, R6A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
